File: pocket-operator-eurorack/pocket-operator-eurorack.sch (KiCad schematic (older format))
At the start: 23 parts

Commit message: front silkscreen artwork finished
Parts:
- added D? (x2): LED, symbol Device:LED
- added R? (x2): R, symbol Device:R
- gave numbers to parts that had none: 23
Connections:
- net GND: now also R?.2, R?.2
- net at J4.S, J8.1 (Pin_1): now also D?.1 (K)
- new net: D?.2 (A), R?.1 (x2)
Other:
- moved on the sheet: J6, J8
